File: Circuit/CanSat/BNO085.kicad_sch (KiCad schematic)
At the start: 10 parts, among them U23 BNO085, U7 ASEK-32.768KHZ-L-R-T

Commit message: pcb last before finish
Connections:
- net 3V3 is gone; now on net +3.3V: R97.2
Changed lines of the file:
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@@
 		)
 	)
-	(hierarchical_label "3V3"
-		(shape input)
+	(global_label "+3.3V"
+		(shape output)
 		(at 142.24 80.01 0)
+		(fields_autoplaced yes)
 		(effects
 			(font
@@
 			(justify left)
 		)
+		(property "Intersheetrefs" "${INTERSHEET_REFS}"
+			(at 151.0051 80.01 0)
+			(effects
+				(font
+					(size 1.27 1.27)
+				)
+				(justify left)
+				(hide yes)
+			)
+		)
 	)
