File: Circuit/CanSat/CanSat.kicad_pcb (KiCad board)
At the start: 4 copper layers, 60 x 60 mm, 108 parts, among them IC1 TPS61088RHLT, J1 GPS, J12 USB_C, J2 Battery, J3 FLIR, J4 2.4G_Radio, J5 Conn_01x07_Pin, J6 Conn_01x06_Socket, Q1 BC817, Q2 BC817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

Commit message: pcb last before finish
Parts:
- added J7: Conn_01x06_Socket, Connector_PinHeader_2.54mm:PinHeader_1x06_P2.54mm_Vertical, F.Cu at (109.2, 114.8)
- C6: moved to B.Cu
- J2: value Battery -> Conn_01x02_Socket; footprint Connector_JST:JST_PH_B3B-PH-K_1x03_P2.00mm_Vertical -> Connector_JST:JST_PH_B2B-PH-K_1x02_P2.00mm_Vertical; moved to F.Cu
- moved C47 44.4 mm to (102.2, 114.2), turned to 90 degrees
- moved C46 42.2 mm to (100.2, 114.2), turned to 90 degrees
- moved C44 40.3 mm to (98.2, 114.2), turned to 90 degrees
- moved C34 38.5 mm to (96.2, 114.2), turned to 90 degrees
- moved C6 35.6 mm to (92.9, 87.9), turned to -90 degrees
- moved J2 3.45 mm to (89.0, 122.6), turned to 0 degrees
- moved C16 0.20 mm to (86.0, 119.8)
- turned L2 to -90 degrees
Connections:
- C11 pad 1: GND -> /PSU/Input-Voltage
- C12 pad 1: GND -> /PSU/Input-Voltage
- C17 pad 2: Net-(C17-Pad2) -> GND
- C21 pad 2: Net-(C17-Pad2) -> GND
- C22 pad 2: Net-(C17-Pad2) -> GND
- C24 pad 2: Net-(C17-Pad2) -> GND
- C34 pad 2: Net-(C34-Pad2) -> GND
- C44 pad 2: Net-(C34-Pad2) -> GND
- C46 pad 2: Net-(C34-Pad2) -> GND
- C47 pad 2: Net-(C34-Pad2) -> GND
- IC1 pad 2: GND -> /PSU/Input-Voltage
- IC1 pad 9: GND -> /PSU/Input-Voltage
- J2 pad 1: unconnected-(J2-Pin_1-Pad1) -> /PSU/Input-Voltage
- J2 pad 2: unconnected-(J2-Pin_2-Pad2) -> GND
- L2 pad 1: GND -> Net-(IC1-SW_1)
- L2 pad 2: Net-(IC1-SW_1) -> /PSU/Input-Voltage
- R97 pad 2: /BNO085/3V3 -> +3.3V
- U3 pad 18: /ESP32-S3-WROOM-1/433Mhz_AUX -> /AUX
- U3 pad 24: /ESP32-S3-WROOM-1/433Mhz_M1 -> /M1
- U3 pad 25: /ESP32-S3-WROOM-1/433Mhz_M0 -> /M0
- U3 pad 26: unconnected-(U3-IO45-Pad26) -> /sd_cs
- U3 pad 34: /ESP32-S3-WROOM-1/433Mhz_ESP_TX -> /RX
- U3 pad 35: /ESP32-S3-WROOM-1/433Mhz_ESP_RX -> /TX
- U4 pad 2: GND -> /PSU/Input-Voltage
- U4 pad 3: GND -> /PSU/Input-Voltage
Routing:
- net /SPI_MISO: track 17.3 -> 85.9 mm, vias 1 -> 3
- net /SPI_CLK: track 14.9 -> 74.3 mm, vias 1 -> 3
- net +3.3V: track 219.7 -> 276.0 mm, vias 5 -> 6
- net /2.4g_cs: track 0.00 -> 49.3 mm, vias 0 -> 1
- net /SPI_MOSI: track 17.7 -> 66.5 mm, vias 1 -> 3
- net /2.4g_int: track 0.00 -> 48.6 mm
- net /GPS_RX: track 0.00 -> 43.1 mm, vias 0 -> 1
- net /RX: track 0.00 -> 42.9 mm, vias 0 -> 1
- net /GPS_TX: track 0.00 -> 41.6 mm, vias 0 -> 1
- net /bno_rst: track 3.98 -> 43.9 mm, vias 0 -> 3
- net /M0: track 0.00 -> 38.6 mm, vias 0 -> 1
- net /M1: track 0.00 -> 38.1 mm, vias 0 -> 1
- net /TX: track 0.00 -> 37.2 mm, vias 0 -> 1
- net /PSU/Input-Voltage: track 0.00 -> 36.7 mm, vias 0 -> 1
- net /2.4g_en: track 0.00 -> 33.3 mm
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- added copper zone on B.Cu, net /PSU/Input-Voltage
