File: Circuit/CanSat/CanSat.kicad_pcb (KiCad board)
At the start: 4 copper layers, 60 x 60 mm, 110 parts, among them IC1 TPS61088RHLT, J1 GPS, J12 USB_C, J3 FLIR, J4 2.4G_Radio, J5 Conn_01x07_Pin, J6 Conn_01x06_Socket, J7 Conn_01x06_Socket, J8 GPS, Q1 BC817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

Commit message: latest pcb, sx module, initial new sensor panel
Parts:
- added R13: 10k, Resistor_SMD:R_0805_2012Metric, F.Cu at (112.8, 75.4)
- added R14: 10k, Resistor_SMD:R_0805_2012Metric, F.Cu at (110.8, 75.4)
- added R15: 0R, Resistor_SMD:R_0805_2012Metric, F.Cu at (78.5, 106.8)
- Battery, C16: moved to B.Cu
- C14: value 68pf -> 10nf
- R3, R6: value 105k -> 300k
- moved C16 4.20 mm to (86.0, 124.0), turned to 180 degrees
- moved C2 0.21 mm to (92.8, 79.3)
Connections:
- IC1 pad 13: unconnected-(IC1-MODE-Pad13) -> Net-(IC1-MODE)
- U1 pad 1: /Slow-SDA -> /Slow-SCL
- U1 pad 4: /Slow-SCL -> /Slow-SDA
- U14 pad 1: unconnected-(U14-A1-Pad1) -> /Slow-SCL
- U14 pad 2: unconnected-(U14-A0-Pad2) -> /Slow-SCL
- U2 pad 3: /SGP41/SDA -> /Slow-SDA
- U2 pad 6: /SGP41/SCL -> /Slow-SCL
- U21 pad 3: /Slow-SCL -> /Slow-SDA
- U21 pad 4: /Slow-SDA -> /Slow-SCL
- U5 pad 1: unconnected-(U5-A1-Pad1) -> /Slow-SDA
- U5 pad 2: unconnected-(U5-A0-Pad2) -> /Slow-SDA
Routing:
- net Net-(IC1-MODE): track 0.00 -> 9.24 mm, vias 0 -> 1
- net +3.3V: track 281.3 -> 289.2 mm, vias 6 -> 7
- net Net-(U14-Vbus): track 33.7 -> 30.8 mm
- net /Slow-SDA: track 88.3 -> 90.0 mm
- net /Slow-SCL: track 99.6 -> 101.0 mm
Other:
- board text added: "#Jedlik"
- board text added: "V1.4.5"
