File: Circuit/CanSat/ESP32-S3-WROOM-1.kicad_sch (KiCad schematic)
At the start: 18 parts, among them J12 USB_C, Q1 BC817, Q2 BC817, U3 ESP32-S3-WROOM-1, U8 CH340G, Y2 12MHz

Commit message: pcb last before finish
Connections:
- net sd_cs: now reaches U3.26 (IO45)
- no-connect marks 5 -> 13
Changed lines of the file:
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@@
 	)
 	(no_connect
-		(at 176.53 58.42)
+		(at 76.2 58.42)
+	)
+	(no_connect
+		(at 45.72 50.8)
+	)
+	(no_connect
+		(at 176.53 59.69)
 	)
 	(no_connect
@@
 	)
 	(no_connect
+		(at 76.2 48.26)
+	)
+	(no_connect
 		(at 196.85 63.5)
+	)
+	(no_connect
+		(at 76.2 60.96)
+	)
+	(no_connect
+		(at 76.2 78.74)
+	)
+	(no_connect
+		(at 76.2 55.88)
+	)
+	(no_connect
+		(at 76.2 50.8)
+	)
+	(no_connect
+		(at 76.2 53.34)
 	)
 	(wire
@@
 		)
 	)
+	(hierarchical_label "sd_cs"
+		(shape input)
+		(at 76.2 76.2 0)
+		(effects
+			(font
+				(size 1.27 1.27)
+			)
+			(justify left)
+		)
+	)

Commit message: latest pcb, sx module, initial new sensor panel
Connections:
- no-connect marks 13 -> 15
Changed lines of the file:
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@@
+	)
+	(no_connect
+		(at 161.29 76.2)
+	)
+	(no_connect
+		(at 161.29 78.74)
 	)
 	(no_connect
