File: Circuit/CanSat/PSU.kicad_sch (KiCad schematic)
At the start: 51 parts, among them IC1 TPS61088RHLT, U14 INA226, U4 AP64501SP-13, U5 INA226

Commit message: pcb last before finish
Connections:
- net GND: now also C17.2, C21.2, C22.2, C24.2, C34.2, C44.2, C46.2, C47.2; no longer C11.1, C12.1, IC1.2 (EN), IC1.9 (VIN), L2.1, U4.2 (VIN), U4.3 (EN)
- net at C10.1, IC1.4 (SW_1), IC1.5 (SW_2)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: now also L2.1; no longer L2.2
- new net Input-Voltage: C11.1, C12.1, IC1.2 (EN), IC1.9 (VIN), L2.2, U4.2 (VIN), U4.3 (EN)
Other:
- note added: "10n el ment a roboton"
- moved on the sheet: C2, C25, C26, C3, C31, C33, L2, R28

Commit message: latest pcb, sx module, initial new sensor panel
Parts:
- added R15: 0R, Resistor_SMD:R_0805_2012Metric, symbol Device:R
- C14: value 68pf -> 10nf
- R3, R6: value 105k -> 300k
Connections:
- net GND: now also R15.1
- net SCL: now also U14.1 (A1), U14.2 (A0)
- net SDA: now also U5.1 (A1), U5.2 (A0)
- net at IC1.13 (MODE): now also R15.2
Other:
- note added: "100 uf ek és 82 mohm"
- note added: "4B"
- note added: "4F"
- moved on the sheet: C31, C33
