File: Circuit/CanSat_V2/CanSat.kicad_pcb (KiCad board)
At the start: 2 copper layers, 24 parts, among them IC1 E22-900M22S, IC2 ZMOD4410AI1V, J1 FLIR_Lepton_Molex_1050281001, SW1 SKRHABE010, U1 AD7091R-8BCPZ-RL7, U10 SCD41-D-R2, U11 SGP41-D-R4, U12 SHT41-AD1B-R2, U13 SIM7080G, U14 STC31-C-R3, U15 VEML7700-TT, U2 AS7331-AQFM, U3 ADS1220IPWR, U4 BME280, U5 BME688, U6 ESP32-P4-Module, U7 LC86G, U8 MICS-6814, U9 RadNano

Commit message: first cansat V2 commit
Parts:
- removed J1: FLIR_Lepton_Molex_1050281001, panel:flir_CONN_1050282031_MOL
- added C1: 100nF, Capacitor_SMD:C_0603_1608Metric_Pad1.08x0.95mm_HandSolder, F.Cu at (14.7, 37.1)
- added C10: 4.7uF, Capacitor_SMD:C_1206_3216Metric, F.Cu at (51.6, 24.1)
- added C100: 4.7uF, Capacitor_SMD:C_1206_3216Metric, F.Cu at (309.9, 58.2)
- added C101: 4.7uF, Capacitor_SMD:C_1206_3216Metric, F.Cu at (309.9, 61.5)
- added C102: 4.7uF, Capacitor_SMD:C_1206_3216Metric, F.Cu at (309.9, 64.9)
- added C103: 4.7uF, Capacitor_SMD:C_1206_3216Metric, F.Cu at (309.9, 68.2)
- added C104: 4.7uF, Capacitor_SMD:C_1206_3216Metric, F.Cu at (309.9, 71.6)
- added C105: 4.7uF, Capacitor_SMD:C_1206_3216Metric, F.Cu at (309.9, 74.9)
- added C106: 4.7uF, Capacitor_SMD:C_1206_3216Metric, F.Cu at (309.9, 78.3)
- added C107: 100nF, Capacitor_SMD:C_0603_1608Metric_Pad1.08x0.95mm_HandSolder, F.Cu at (-234.5, -55.6)
- added C108: 100nF, Capacitor_SMD:C_0603_1608Metric_Pad1.08x0.95mm_HandSolder, F.Cu at (-234.5, -53.1)
- added C109: 100nF, Capacitor_SMD:C_0603_1608Metric_Pad1.08x0.95mm_HandSolder, F.Cu at (-234.5, -50.6)
- added C11: 4.7uF, Capacitor_SMD:C_1206_3216Metric, F.Cu at (51.6, 27.5)
- added C110: 100nF, Capacitor_SMD:C_0603_1608Metric_Pad1.08x0.95mm_HandSolder, F.Cu at (-234.5, -48.1)
- added C111: 100nF, Capacitor_SMD:C_0603_1608Metric_Pad1.08x0.95mm_HandSolder, F.Cu at (-234.5, -45.6)
- added C112: 4.7uF, Capacitor_SMD:C_1206_3216Metric, F.Cu at (-204.4, -41.4)
- added C113: 4.7uF, Capacitor_SMD:C_1206_3216Metric, F.Cu at (-204.4, -38.1)
- added C114: 100nF, Capacitor_SMD:C_0603_1608Metric_Pad1.08x0.95mm_HandSolder, F.Cu at (-209.4, -41.9)
- added C115: 100nF, Capacitor_SMD:C_0603_1608Metric_Pad1.08x0.95mm_HandSolder, F.Cu at (-209.4, -39.4)
- added C116: 4.7uF, Capacitor_SMD:C_1206_3216Metric, F.Cu at (-204.4, -34.7)
- added C117: 4.7uF, Capacitor_SMD:C_1206_3216Metric, F.Cu at (-204.4, -31.4)
- added C118: 100nF, Capacitor_SMD:C_0603_1608Metric_Pad1.08x0.95mm_HandSolder, F.Cu at (-209.6, -65.6)
- added C119: 100nF, Capacitor_SMD:C_0603_1608Metric_Pad1.08x0.95mm_HandSolder, F.Cu at (-209.6, -63.1)
- added C12: 100nF, Capacitor_SMD:C_0603_1608Metric_Pad1.08x0.95mm_HandSolder, F.Cu at (46.6, 10.8)
- added C120: 4.7uF, Capacitor_SMD:C_1206_3216Metric, F.Cu at (-195.9, -48.4)
- added C121: 10pF, Capacitor_SMD:C_0402_1005Metric_Pad0.74x0.62mm_HandSolder, F.Cu at (-205.6, -50.8)
- added C122: 47pF, Capacitor_SMD:C_0402_1005Metric_Pad0.74x0.62mm_HandSolder, F.Cu at (-205.6, -48.8)
- added C123: 100nF, Capacitor_SMD:C_0603_1608Metric_Pad1.08x0.95mm_HandSolder, F.Cu at (-209.6, -60.6)
- added C124: 100nF, Capacitor_SMD:C_0603_1608Metric_Pad1.08x0.95mm_HandSolder, F.Cu at (-209.6, -58.0)
- added C125: 100nF, Capacitor_SMD:C_0603_1608Metric_Pad1.08x0.95mm_HandSolder, F.Cu at (-209.6, -55.5)
- added C126: 1nF, Capacitor_SMD:C_0402_1005Metric_Pad0.74x0.62mm_HandSolder, F.Cu at (-205.6, -46.8)
- added C127: 100nF, Capacitor_SMD:C_0603_1608Metric_Pad1.08x0.95mm_HandSolder, F.Cu at (-238.8, -41.1)
- added C128: 4.7uF, Capacitor_SMD:C_1206_3216Metric, F.Cu at (-225.1, -40.6)
- added C129: 4.7uF, Capacitor_SMD:C_1206_3216Metric, F.Cu at (-225.1, -37.3)
- added C13: 100nF, Capacitor_SMD:C_0603_1608Metric_Pad1.08x0.95mm_HandSolder, F.Cu at (46.6, 13.3)
- added C130: 100nF, Capacitor_SMD:C_0603_1608Metric_Pad1.08x0.95mm_HandSolder, F.Cu at (-238.8, -38.6)
- added C131: 100nF, Capacitor_SMD:C_0603_1608Metric_Pad1.08x0.95mm_HandSolder, F.Cu at (-238.8, -36.0)
- added C132: 1pF, Capacitor_SMD:C_0402_1005Metric_Pad0.74x0.62mm_HandSolder, F.Cu at (-220.7, -41.3)
- added C133: 4.7uF, Capacitor_SMD:C_1206_3216Metric, F.Cu at (-225.1, -34.0)
- added C134: 15pF, Capacitor_SMD:C_0402_1005Metric_Pad0.74x0.62mm_HandSolder, F.Cu at (-220.7, -39.4)
- added C135: 100nF, Capacitor_SMD:C_0603_1608Metric_Pad1.08x0.95mm_HandSolder, F.Cu at (-238.8, -33.5)
- added C136: 100nF, Capacitor_SMD:C_0603_1608Metric_Pad1.08x0.95mm_HandSolder, F.Cu at (-238.8, -31.0)
- added C137: 100nF, Capacitor_SMD:C_0603_1608Metric_Pad1.08x0.95mm_HandSolder, F.Cu at (-238.8, -28.5)
- added C138: 1nF, Capacitor_SMD:C_0402_1005Metric_Pad0.74x0.62mm_HandSolder, F.Cu at (-220.7, -37.4)
- added C139: 4.7uF, Capacitor_SMD:C_1206_3216Metric, F.Cu at (-225.1, -30.6)
- added C14: 22uF, Capacitor_SMD:C_1210_3225Metric, F.Cu at (57.3, 26.0)
- added C140: 4.7uF, Capacitor_SMD:C_1206_3216Metric, F.Cu at (-225.1, -27.2)
- added C141: 4.7uF, Capacitor_SMD:C_1206_3216Metric, F.Cu at (-89.0, -56.0)
- added C142: 4.7uF, Capacitor_SMD:C_1206_3216Metric, F.Cu at (-89.0, -52.6)
- added C143: 4.7uF, Capacitor_SMD:C_1206_3216Metric, F.Cu at (-89.0, -49.3)
- added C144: 4.7uF, Capacitor_SMD:C_1206_3216Metric, F.Cu at (-89.0, -45.9)
- added C145: 4.7uF, Capacitor_SMD:C_1206_3216Metric, F.Cu at (-89.0, -42.6)
- added C146: 4.7uF, Capacitor_SMD:C_1206_3216Metric, F.Cu at (-89.0, -39.2)
- added C147: 100nF, Capacitor_SMD:C_0603_1608Metric_Pad1.08x0.95mm_HandSolder, F.Cu at (-70.2, -48.7)
- added C148: 100nF, Capacitor_SMD:C_0603_1608Metric_Pad1.08x0.95mm_HandSolder, F.Cu at (-70.2, -46.2)
- added C149: 100nF, Capacitor_SMD:C_0603_1608Metric_Pad1.08x0.95mm_HandSolder, F.Cu at (-70.2, -43.7)
- added C15: 4.7uF, Capacitor_SMD:C_1206_3216Metric, F.Cu at (101.2, 9.63)
- added C16: 4.7uF, Capacitor_SMD:C_1206_3216Metric, F.Cu at (101.2, 13.0)
- added C17: 4.7uF, Capacitor_SMD:C_1206_3216Metric, F.Cu at (101.2, 16.3)
- added C18: 4.7uF, Capacitor_SMD:C_1206_3216Metric, F.Cu at (101.2, 19.7)
- added C19: 100nF, Capacitor_SMD:C_0603_1608Metric_Pad1.08x0.95mm_HandSolder, F.Cu at (46.6, -13.7)
- added C2: 100nF, Capacitor_SMD:C_0603_1608Metric_Pad1.08x0.95mm_HandSolder, F.Cu at (13.9, 40.2)
- added C20: 100nF, Capacitor_SMD:C_0603_1608Metric_Pad1.08x0.95mm_HandSolder, F.Cu at (46.6, -11.2)
- added C21: 100nF, Capacitor_SMD:C_0603_1608Metric_Pad1.08x0.95mm_HandSolder, F.Cu at (46.6, -8.70)
- added C22: 100nF, Capacitor_SMD:C_0603_1608Metric_Pad1.08x0.95mm_HandSolder, F.Cu at (43.8, 51.5)
- added C23: 22uF, Capacitor_SMD:C_1210_3225Metric, F.Cu at (44.5, 64.9)
- added C24: 100nF, Capacitor_SMD:C_0603_1608Metric_Pad1.08x0.95mm_HandSolder, F.Cu at (43.8, 54.0)
- added C25: 100nF, Capacitor_SMD:C_0603_1608Metric_Pad1.08x0.95mm_HandSolder, F.Cu at (43.8, 56.5)
- added C26: 100nF, Capacitor_SMD:C_0603_1608Metric_Pad1.08x0.95mm_HandSolder, F.Cu at (43.8, 59.0)
- added C27: 22uF, Capacitor_SMD:C_1210_3225Metric, F.Cu at (44.5, 69.1)
- added C28: 22pF, Capacitor_SMD:C_0402_1005Metric_Pad0.74x0.62mm_HandSolder, F.Cu at (90.8, 38.9)
- added C29: 22pF, Capacitor_SMD:C_0402_1005Metric_Pad0.74x0.62mm_HandSolder, F.Cu at (90.8, 40.8)
- added C3: 22uF, Capacitor_SMD:C_1210_3225Metric, F.Cu at (74.5, 35.2)
- added C30: 100nF, Capacitor_SMD:C_0603_1608Metric_Pad1.08x0.95mm_HandSolder, F.Cu at (91.3, 31.6)
- added C31: 100nF, Capacitor_SMD:C_0603_1608Metric_Pad1.08x0.95mm_HandSolder, F.Cu at (91.3, 34.1)
- added C32: 100nF, Capacitor_SMD:C_0603_1608Metric_Pad1.08x0.95mm_HandSolder, F.Cu at (91.3, 36.6)
- added C33: 100nF, Capacitor_SMD:C_0603_1608Metric_Pad1.08x0.95mm_HandSolder, F.Cu at (156.0, 132.6)
- added C34: 100nF, Capacitor_SMD:C_0603_1608Metric_Pad1.08x0.95mm_HandSolder, F.Cu at (156.0, 135.1)
- added C35: 22uF, Capacitor_SMD:C_1210_3225Metric, F.Cu at (151.0, 133.4)
- added C36: 22uF, Capacitor_SMD:C_1210_3225Metric, F.Cu at (151.0, 137.7)
- added C37: 100nF, Capacitor_SMD:C_0603_1608Metric_Pad1.08x0.95mm_HandSolder, F.Cu at (156.0, 137.6)
- added C38: 100nF, Capacitor_SMD:C_0603_1608Metric_Pad1.08x0.95mm_HandSolder, F.Cu at (156.0, 140.1)
- added C39: 22uF, Capacitor_SMD:C_1210_3225Metric, F.Cu at (151.0, 141.9)
- added C4: 100nF, Capacitor_SMD:C_0603_1608Metric_Pad1.08x0.95mm_HandSolder, F.Cu at (69.5, 34.3)
- added C40: 22uF, Capacitor_SMD:C_1210_3225Metric, F.Cu at (151.0, 146.2)
- added C41: 22uF, Capacitor_SMD:C_1210_3225Metric, F.Cu at (151.0, 150.4)
- added C42: -, Capacitor_SMD:C_0402_1005Metric_Pad0.74x0.62mm_HandSolder, F.Cu at (141.5, 133.0)
- added C43: -, Capacitor_SMD:C_0402_1005Metric_Pad0.74x0.62mm_HandSolder, F.Cu at (141.5, 135.0)
- added C44: -, Capacitor_SMD:C_0402_1005Metric_Pad0.74x0.62mm_HandSolder, F.Cu at (141.5, 136.9)
- added C45: -, Capacitor_SMD:C_0402_1005Metric_Pad0.74x0.62mm_HandSolder, F.Cu at (141.5, 138.9)
- added C46: 100nF, Capacitor_SMD:C_0603_1608Metric_Pad1.08x0.95mm_HandSolder, F.Cu at (123.4, 133.3)
- added C47: 100nF, Capacitor_SMD:C_0603_1608Metric_Pad1.08x0.95mm_HandSolder, F.Cu at (123.4, 135.8)
- added C48: 22uF, Capacitor_SMD:C_1210_3225Metric, F.Cu at (137.1, 134.2)
- added C49: 22uF, Capacitor_SMD:C_1210_3225Metric, F.Cu at (137.1, 138.4)
- added C5: 100nF, Capacitor_SMD:C_0603_1608Metric_Pad1.08x0.95mm_HandSolder, F.Cu at (69.5, 17.3)
- added C50: 100nF, Capacitor_SMD:C_0603_1608Metric_Pad1.08x0.95mm_HandSolder, F.Cu at (123.4, 138.3)
- added C51: 4.7uF, Capacitor_SMD:C_1206_3216Metric, F.Cu at (305.1, 98.5)
- added C52: 4.7uF, Capacitor_SMD:C_1206_3216Metric, F.Cu at (305.1, 101.9)
- added C53: 100nF, Capacitor_SMD:C_0603_1608Metric_Pad1.08x0.95mm_HandSolder, F.Cu at (289.6, 88.5)
- added C54: 100nF, Capacitor_SMD:C_0603_1608Metric_Pad1.08x0.95mm_HandSolder, F.Cu at (289.6, 91.0)
- added C55: 100nF, Capacitor_SMD:C_0603_1608Metric_Pad1.08x0.95mm_HandSolder, F.Cu at (289.6, 93.5)
- added C56: 100nF, Capacitor_SMD:C_0603_1608Metric_Pad1.08x0.95mm_HandSolder, F.Cu at (289.6, 96.0)
- added C57: 4.7uF, Capacitor_SMD:C_1206_3216Metric, F.Cu at (272.7, 49.5)
- added C58: 4.7uF, Capacitor_SMD:C_1206_3216Metric, F.Cu at (272.7, 52.9)
- added C59: 4.7uF, Capacitor_SMD:C_1206_3216Metric, F.Cu at (272.7, 56.2)
- added C6: 100nF, Capacitor_SMD:C_0603_1608Metric_Pad1.08x0.95mm_HandSolder, F.Cu at (69.5, 19.8)
- added C60: 4.7uF, Capacitor_SMD:C_1206_3216Metric, F.Cu at (272.7, 59.5)
- added C61: 4.7uF, Capacitor_SMD:C_1206_3216Metric, F.Cu at (272.7, 62.9)
- added C62: 4.7uF, Capacitor_SMD:C_1206_3216Metric, F.Cu at (272.7, 66.2)
- added C63: 4.7uF, Capacitor_SMD:C_1206_3216Metric, F.Cu at (272.7, 69.6)
- added C64: 4.7uF, Capacitor_SMD:C_1206_3216Metric, F.Cu at (272.7, 73.0)
- added C65: 100nF, Capacitor_SMD:C_0603_1608Metric_Pad1.08x0.95mm_HandSolder, F.Cu at (277.7, 49.1)
- added C66: 22uF, Capacitor_SMD:C_1210_3225Metric, F.Cu at (282.7, 68.3)
- added C67: 22uF, Capacitor_SMD:C_1210_3225Metric, F.Cu at (282.7, 72.6)
- added C68: 100nF, Capacitor_SMD:C_0603_1608Metric_Pad1.08x0.95mm_HandSolder, F.Cu at (187.6, 50.2)
- added C69: 10nF, Capacitor_SMD:C_0603_1608Metric_Pad1.08x0.95mm_HandSolder, F.Cu at (187.6, 52.7)
- added C7: 100nF, Capacitor_SMD:C_0603_1608Metric_Pad1.08x0.95mm_HandSolder, F.Cu at (69.5, 22.3)
- added C70: 68pF, Capacitor_SMD:C_0402_1005Metric_Pad0.74x0.62mm_HandSolder, F.Cu at (191.4, 59.5)
- added C71: 1.2nF, Capacitor_SMD:C_0805_2012Metric_Pad1.18x1.45mm_HandSolder, F.Cu at (192.2, 57.1)
- added C72: 68pF, Capacitor_SMD:C_0402_1005Metric_Pad0.74x0.62mm_HandSolder, F.Cu at (191.4, 61.5)
- added C73: 22uF, Capacitor_SMD:C_1210_3225Metric, F.Cu at (182.6, 43.0)
- added C74: 22uF, Capacitor_SMD:C_1210_3225Metric, F.Cu at (182.6, 47.2)
- added C75: 22uF, Capacitor_SMD:C_1210_3225Metric, F.Cu at (182.6, 51.5)
- added C76: 22uF, Capacitor_SMD:C_1210_3225Metric, F.Cu at (182.6, 55.7)
- added C77: 22uF, Capacitor_SMD:C_1210_3225Metric, F.Cu at (182.6, 60.0)
- added C78: 22uF, Capacitor_SMD:C_1210_3225Metric, F.Cu at (182.6, 64.2)
- added C79: 4.7uF, Capacitor_SMD:C_1206_3216Metric, F.Cu at (235.4, 20.4)
- added C8: 100nF, Capacitor_SMD:C_0603_1608Metric_Pad1.08x0.95mm_HandSolder, F.Cu at (69.5, 24.8)
- added C80: 4.7uF, Capacitor_SMD:C_1206_3216Metric, F.Cu at (235.4, 23.8)
- added C81: 4.7uF, Capacitor_SMD:C_1206_3216Metric, F.Cu at (235.4, 27.1)
- added C82: 4.7uF, Capacitor_SMD:C_1206_3216Metric, F.Cu at (235.4, 30.5)
- added C83: 4.7uF, Capacitor_SMD:C_1206_3216Metric, F.Cu at (235.4, 33.9)
- added C84: 4.7uF, Capacitor_SMD:C_1206_3216Metric, F.Cu at (241.1, 20.4)
- added C85: 22uF, Capacitor_SMD:C_1210_3225Metric, F.Cu at (229.8, 20.9)
- added C86: 22uF, Capacitor_SMD:C_1210_3225Metric, F.Cu at (229.8, 25.1)
- added C87: 4.7uF, Capacitor_SMD:C_1206_3216Metric, F.Cu at (241.1, 23.8)
- added C88: 4.7uF, Capacitor_SMD:C_1206_3216Metric, F.Cu at (241.1, 27.1)
- added C89: 4.7uF, Capacitor_SMD:C_1206_3216Metric, F.Cu at (241.1, 30.5)
- added C9: 4.7uF, Capacitor_SMD:C_1206_3216Metric, F.Cu at (51.6, 20.8)
- added C90: 4.7uF, Capacitor_SMD:C_1206_3216Metric, F.Cu at (241.1, 33.9)
- added C91: 4.7uF, Capacitor_SMD:C_1206_3216Metric, F.Cu at (246.7, 20.4)
- added C92: 4.7uF, Capacitor_SMD:C_1206_3216Metric, F.Cu at (246.7, 23.8)
- added C93: 22uF, Capacitor_SMD:C_1210_3225Metric, F.Cu at (229.8, 29.4)
- added C94: 22uF, Capacitor_SMD:C_1210_3225Metric, F.Cu at (229.8, 33.6)
- added C95: 4.7uF, Capacitor_SMD:C_1206_3216Metric, F.Cu at (246.7, 27.1)
- added C96: 4.7uF, Capacitor_SMD:C_1206_3216Metric, F.Cu at (246.7, 30.5)
- added C97: 4.7uF, Capacitor_SMD:C_1206_3216Metric, F.Cu at (246.7, 33.9)
- added C98: 22uF, Capacitor_SMD:C_1210_3225Metric, F.Cu at (229.8, 37.9)
- added C99: 4.7uF, Capacitor_SMD:C_1206_3216Metric, F.Cu at (309.9, 54.8)
- added CN1: 61082-041402LF, panel:CONN-SMD_61082-041402LF, F.Cu at (9.10, 18.5)
- added CN2: 61082-041402LF, panel:CONN-SMD_61082-041402LF, F.Cu at (163.0, 97.8)
- added D1: LED, LED_SMD:LED_0603_1608Metric_Pad1.05x0.95mm_HandSolder, F.Cu at (22.8, 14.8)
- added D10: LED, LED_SMD:LED_0603_1608Metric_Pad1.05x0.95mm_HandSolder, F.Cu at (195.2, 59.9)
- added D11: BAT54J, Diode_SMD:D_SOD-323_HandSoldering, F.Cu at (-204.7, -23.9)
- added D12: SiPM, panel:OPTO-SMD_4P-MICROFC-60035-SMT-TR, F.Cu at (-194.6, -62.6)
- added D13: TECH PUBLIC BAS70WS, Diode_SMD:D_SOD-323_HandSoldering, F.Cu at (-201.4, -50.3)
- added D14: SiPM, panel:OPTO-SMD_4P-MICROFC-60035-SMT-TR, F.Cu at (-223.7, -21.4)
- added D15: TECH PUBLIC BAS70WS, Diode_SMD:D_SOD-323_HandSoldering, F.Cu at (-238.4, -23.3)
- added D2: LED, LED_SMD:LED_0603_1608Metric_Pad1.05x0.95mm_HandSolder, F.Cu at (22.8, 17.4)
- added D3: LED, LED_SMD:LED_0603_1608Metric_Pad1.05x0.95mm_HandSolder, F.Cu at (73.9, 38.6)
- added D4: LED, LED_SMD:LED_0603_1608Metric_Pad1.05x0.95mm_HandSolder, F.Cu at (63.2, -1.13)
- added D5: LED, LED_SMD:LED_0603_1608Metric_Pad1.05x0.95mm_HandSolder, F.Cu at (63.2, 1.46)
- added D6: ESD5311X-2/TR, Diode_SMD:D_0402_1005Metric_Pad0.77x0.64mm_HandSolder, F.Cu at (127.6, 149.8)
- added D7: ESD5311X-2/TR, Diode_SMD:D_0402_1005Metric_Pad0.77x0.64mm_HandSolder, F.Cu at (127.6, 151.8)
- added D8: LED, LED_SMD:LED_0603_1608Metric_Pad1.05x0.95mm_HandSolder, F.Cu at (132.3, 148.4)
- added D9: LED, LED_SMD:LED_0603_1608Metric_Pad1.05x0.95mm_HandSolder, F.Cu at (132.3, 151.0)
- added FB1: FerriteBead_Small, Diode_SMD:D_0805_2012Metric, F.Cu at (-199.3, -32.9)
- added FB2: FerriteBead_Small, Diode_SMD:D_0805_2012Metric, F.Cu at (-199.3, -29.9)
- added FPC1: 61083-044402LF, panel:FPC-SMD_40P-P0.80_61083-044402LF, B.Cu at (105.7, 97.8)
- added FPC2: 61083-044402LF, panel:FPC-SMD_40P-P0.80_61083-044402LF, F.Cu at (255.2, 100.3)
- added IC3: E22-xxxM22S, panel:E22-400M22S, F.Cu at (147.3, 111.3)
- added IC4: E22-xxxM22S, panel:E22-400M22S, B.Cu at (147.1, 85.4)
- added J10: VTX PWR, Connector_JST:JST_PH_B4B-PH-K_1x04_P2.00mm_Vertical, F.Cu at (238.2, 99.3)
- added J11: GLM-670, Connector_Wire:SolderWire-0.127sqmm_1x04_P3.7mm_D0.48mm_OD1mm_Relief, F.Cu at (293.7, 89.1)
- added J12: Conn_01x15_Pin, Connector_FFC-FPC:TE_1-1734839-5_1x15-1MP_P0.5mm_Horizontal, F.Cu at (-229.2, -61.6)
- added J13: Conn_01x15_Pin, Connector_FFC-FPC:TE_1-1734839-5_1x15-1MP_P0.5mm_Horizontal, F.Cu at (-78.7, -54.7)
- added J14: FLIR_Lepton_Molex_1050281001, panel:flir_CONN_1050282031_MOL, F.Cu at (-79.4, -42.9)
- added J2: Conn_01x15_Pin, Connector_FFC-FPC:TE_1-1734839-5_1x15-1MP_P0.5mm_Horizontal, F.Cu at (5.07, 25.5)
- added J3: Conn_01x15_Pin, Connector_FFC-FPC:TE_1-1734839-5_1x15-1MP_P0.5mm_Horizontal, F.Cu at (5.07, 33.2)
- added J4: USB_C, Connector_USB:USB_C_Receptacle_Palconn_UTC16-G, F.Cu at (74.8, 65.1)
- added J5: USB_C, Connector_USB:USB_C_Receptacle_Palconn_UTC16-G, F.Cu at (86.6, 55.3)
- added J6: USB_C, Connector_USB:USB_C_Receptacle_Palconn_UTC16-G, F.Cu at (86.3, 65.4)
- added J7: U-Fl-IPEX, panel:IPEX-SMD_4P-L2.6-W2.6-LS3.1, F.Cu at (132.6, 144.6)
- added J8: U-Fl-IPEX, panel:IPEX-SMD_4P-L2.6-W2.6-LS3.1, F.Cu at (137.6, 144.6)
- added J9: USB_C, Connector_USB:USB_C_Receptacle_Palconn_UTC16-G, B.Cu at (119.0, 108.8)
- added L1: SMNR4030-1R8MT, Inductor_SMD:L_Taiyo-Yuden_NR-50xx, F.Cu at (50.6, 66.0)
- added L2: FXL0630-3R3-M, Inductor_SMD:L_Bourns_SRP7028A_7.3x6.6mm, F.Cu at (190.4, 44.9)
- added L3: 47uh, Diode_SMD:D_0805_2012Metric, F.Cu at (-199.3, -26.8)
- added Q1: AO3401A, Package_TO_SOT_SMD:SOT-23, F.Cu at (91.6, 10.2)
- added Q10: BC817, Package_TO_SOT_SMD:SOT-23, F.Cu at (288.5, 67.9)
- added Q11: WD070PG, Package_TO_SOT_SMD:SOT-89-3, F.Cu at (283.2, 57.0)
- added Q12: WD070PG, Package_TO_SOT_SMD:SOT-89-3, F.Cu at (283.2, 63.2)
- added Q13: AO3400A, Package_TO_SOT_SMD:SOT-23, F.Cu at (288.5, 72.4)
- added Q14: AO3400A, Package_TO_SOT_SMD:SOT-23, F.Cu at (288.5, 76.8)
- added Q15: AO3401A, Package_TO_SOT_SMD:SOT-23, F.Cu at (233.5, 50.0)
- added Q16: AO3401A, Package_TO_SOT_SMD:SOT-23, F.Cu at (233.5, 54.5)
- added Q17: BC817, Package_TO_SOT_SMD:SOT-23, F.Cu at (233.5, 59.0)
- added Q18: BC817, Package_TO_SOT_SMD:SOT-23, F.Cu at (233.5, 63.4)
- added Q19: AO3401A, Package_TO_SOT_SMD:SOT-23, F.Cu at (233.5, 67.8)
- added Q2: BC817, Package_TO_SOT_SMD:SOT-23, F.Cu at (91.6, 14.6)
- added Q20: AO3401A, Package_TO_SOT_SMD:SOT-23, F.Cu at (238.4, 50.0)
- added Q21: BC817, Package_TO_SOT_SMD:SOT-23, F.Cu at (238.4, 54.5)
- added Q22: BC817, Package_TO_SOT_SMD:SOT-23, F.Cu at (238.4, 59.0)
- added Q23: AO3401A, Package_TO_SOT_SMD:SOT-23, F.Cu at (238.4, 63.4)
- added Q24: BC817, Package_TO_SOT_SMD:SOT-23, F.Cu at (238.4, 67.8)
- added Q25: AO3401A, Package_TO_SOT_SMD:SOT-23, F.Cu at (315.1, 55.4)
- added Q26: BC817, Package_TO_SOT_SMD:SOT-23, F.Cu at (315.1, 59.8)
- added Q27: XNRUSEMI XR2SK3019, Package_TO_SOT_SMD:SOT-523, F.Cu at (-192.1, -56.9)
- added Q28: XNRUSEMI XR2SK3019, Package_TO_SOT_SMD:SOT-523, F.Cu at (-234.0, -19.1)
- added Q3: AO3401A, Package_TO_SOT_SMD:SOT-23, F.Cu at (91.6, 19.1)
- added Q4: BC817, Package_TO_SOT_SMD:SOT-23, F.Cu at (91.6, 23.5)
- added Q5: BC817, Package_TO_SOT_SMD:SOT-23, F.Cu at (58.5, -0.20)
- added Q6: BC817, Package_TO_SOT_SMD:SOT-23, F.Cu at (58.5, 4.25)
- added Q7: BC817, Package_TO_SOT_SMD:SOT-23, F.Cu at (49.7, 71.5)
- added Q8: BC817, Package_TO_SOT_SMD:SOT-23, F.Cu at (136.9, 149.4)
- added Q9: WD070PG, Package_TO_SOT_SMD:SOT-89-3, F.Cu at (283.2, 50.9)
- added R10: 220Ω, Resistor_SMD:R_0603_1608Metric_Pad0.98x0.95mm_HandSolder, F.Cu at (23.4, 39.6)
- added R100: 10kΩ, Resistor_SMD:R_0603_1608Metric_Pad0.98x0.95mm_HandSolder, F.Cu at (257.4, 82.9)
- added R101: shunt, Resistor_SMD:R_0805_2012Metric, F.Cu at (319.2, 70.5)
- added R102: 47kΩ, Resistor_SMD:R_0603_1608Metric_Pad0.98x0.95mm_HandSolder, F.Cu at (314.9, 70.3)
- added R103: 4.7kΩ, Resistor_SMD:R_0603_1608Metric_Pad0.98x0.95mm_HandSolder, F.Cu at (314.9, 72.8)
- added R104: 10kΩ, Resistor_SMD:R_0603_1608Metric_Pad0.98x0.95mm_HandSolder, F.Cu at (314.9, 75.3)
- added R105: shunt, Resistor_SMD:R_0805_2012Metric, F.Cu at (319.2, 73.5)
- added R106: 4.7kΩ, Resistor_SMD:R_0603_1608Metric_Pad0.98x0.95mm_HandSolder, F.Cu at (-230.1, -55.6)
- added R107: 4.7kΩ, Resistor_SMD:R_0603_1608Metric_Pad0.98x0.95mm_HandSolder, F.Cu at (-230.1, -53.1)
- added R108: 4.7kΩ, Resistor_SMD:R_0603_1608Metric_Pad0.98x0.95mm_HandSolder, F.Cu at (-230.1, -50.6)
- added R109: 4.7kΩ, Resistor_SMD:R_0603_1608Metric_Pad0.98x0.95mm_HandSolder, F.Cu at (-230.1, -48.1)
- added R11: 10kΩ, Resistor_SMD:R_0603_1608Metric_Pad0.98x0.95mm_HandSolder, F.Cu at (69.5, 36.8)
- added R110: 4.7kΩ, Resistor_SMD:R_0603_1608Metric_Pad0.98x0.95mm_HandSolder, F.Cu at (-230.1, -45.6)
- added R111: 4.7kΩ, Resistor_SMD:R_0603_1608Metric_Pad0.98x0.95mm_HandSolder, F.Cu at (-225.8, -55.6)
- added R112: 4.7kΩ, Resistor_SMD:R_0603_1608Metric_Pad0.98x0.95mm_HandSolder, F.Cu at (-225.8, -53.1)
- added R113: 4.7kΩ, Resistor_SMD:R_0603_1608Metric_Pad0.98x0.95mm_HandSolder, F.Cu at (-225.8, -50.6)
- added R114: 68kΩ, Resistor_SMD:R_0603_1608Metric_Pad0.98x0.95mm_HandSolder, F.Cu at (-209.4, -36.8)
- added R115: 154kΩ, Resistor_SMD:R_0603_1608Metric_Pad0.98x0.95mm_HandSolder, F.Cu at (-209.4, -34.3)
- added R116: 6,65kΩ, Resistor_SMD:R_0603_1608Metric_Pad0.98x0.95mm_HandSolder, F.Cu at (-209.4, -31.8)
- added R117: 470kΩ, Resistor_SMD:R_0603_1608Metric_Pad0.98x0.95mm_HandSolder, F.Cu at (-209.4, -29.3)
- added R118: 39kΩ, Resistor_SMD:R_0603_1608Metric_Pad0.98x0.95mm_HandSolder, F.Cu at (-209.4, -26.8)
- added R119: 1kΩ, Resistor_SMD:R_0603_1608Metric_Pad0.98x0.95mm_HandSolder, F.Cu at (-209.6, -53.0)
- added R12: 220Ω, Resistor_SMD:R_0603_1608Metric_Pad0.98x0.95mm_HandSolder, F.Cu at (69.5, 39.3)
- added R120: 470Ω, Resistor_SMD:R_0603_1608Metric_Pad0.98x0.95mm_HandSolder, F.Cu at (-205.3, -65.6)
- added R121: 33Ω, Resistor_SMD:R_0603_1608Metric_Pad0.98x0.95mm_HandSolder, F.Cu at (-205.3, -63.1)
- added R122: 10kΩ, Resistor_SMD:R_0603_1608Metric_Pad0.98x0.95mm_HandSolder, F.Cu at (-205.3, -60.6)
- added R123: 1kΩ, Resistor_SMD:R_0603_1608Metric_Pad0.98x0.95mm_HandSolder, F.Cu at (-205.3, -58.0)
- added R124: 4.7kΩ, Resistor_SMD:R_0603_1608Metric_Pad0.98x0.95mm_HandSolder, F.Cu at (-205.3, -55.5)
- added R125: 33Ω, Resistor_SMD:R_0603_1608Metric_Pad0.98x0.95mm_HandSolder, F.Cu at (-205.3, -53.0)
- added R126: 1kΩ, Resistor_SMD:R_0603_1608Metric_Pad0.98x0.95mm_HandSolder, F.Cu at (-200.9, -65.6)
- added R127: 1kΩ, Resistor_SMD:R_0603_1608Metric_Pad0.98x0.95mm_HandSolder, F.Cu at (-200.9, -63.1)
- added R128: 100kΩ, Resistor_SMD:R_0603_1608Metric_Pad0.98x0.95mm_HandSolder, F.Cu at (-200.9, -60.6)
- added R129: 33Ω, Resistor_SMD:R_0603_1608Metric_Pad0.98x0.95mm_HandSolder, F.Cu at (-200.9, -58.0)
- added R13: 18kΩ, Resistor_SMD:R_0603_1608Metric_Pad0.98x0.95mm_HandSolder, F.Cu at (69.5, 27.3)
- added R130: 1kΩ, Resistor_SMD:R_0603_1608Metric_Pad0.98x0.95mm_HandSolder, F.Cu at (-238.8, -26.0)
- added R131: 470Ω, Resistor_SMD:R_0603_1608Metric_Pad0.98x0.95mm_HandSolder, F.Cu at (-234.5, -41.1)
- added R132: 50Ω, Resistor_SMD:R_0603_1608Metric_Pad0.98x0.95mm_HandSolder, F.Cu at (-234.5, -38.6)
- added R133: 100Ω, Resistor_SMD:R_0603_1608Metric_Pad0.98x0.95mm_HandSolder, F.Cu at (-234.5, -36.0)
- added R134: 10kΩ, Resistor_SMD:R_0603_1608Metric_Pad0.98x0.95mm_HandSolder, F.Cu at (-234.5, -33.5)
- added R135: 680Ω, Resistor_SMD:R_0603_1608Metric_Pad0.98x0.95mm_HandSolder, F.Cu at (-234.5, -31.0)
- added R136: 1kΩ, Resistor_SMD:R_0603_1608Metric_Pad0.98x0.95mm_HandSolder, F.Cu at (-234.5, -28.5)
- added R137: 24kΩ, Resistor_SMD:R_0603_1608Metric_Pad0.98x0.95mm_HandSolder, F.Cu at (-234.5, -26.0)
- added R138: 100kΩ, Resistor_SMD:R_0603_1608Metric_Pad0.98x0.95mm_HandSolder, F.Cu at (-230.1, -41.1)
- added R139: 100kΩ, Resistor_SMD:R_0603_1608Metric_Pad0.98x0.95mm_HandSolder, F.Cu at (-230.1, -38.6)
- added R14: 100kΩ, Resistor_SMD:R_0603_1608Metric_Pad0.98x0.95mm_HandSolder, F.Cu at (69.5, 29.8)
- added R140: 150kΩ, Resistor_SMD:R_0603_1608Metric_Pad0.98x0.95mm_HandSolder, F.Cu at (-230.1, -36.0)
- added R141: 100kΩ, Resistor_SMD:R_0603_1608Metric_Pad0.98x0.95mm_HandSolder, F.Cu at (-230.1, -33.5)
- added R142: 33Ω, Resistor_SMD:R_0603_1608Metric_Pad0.98x0.95mm_HandSolder, F.Cu at (-230.1, -31.0)
- added R143: 47kΩ, Resistor_SMD:R_0603_1608Metric_Pad0.98x0.95mm_HandSolder, F.Cu at (-70.2, -41.2)
- added R144: 47kΩ, Resistor_SMD:R_0603_1608Metric_Pad0.98x0.95mm_HandSolder, F.Cu at (23.4, 42.1)
- added R145: 47kΩ, Resistor_SMD:R_0603_1608Metric_Pad0.98x0.95mm_HandSolder, F.Cu at (23.4, 44.6)
- added R15: 20Ω, Resistor_SMD:R_0603_1608Metric_Pad0.98x0.95mm_HandSolder, F.Cu at (46.6, 15.8)
- added R16: 12.4Ω, Resistor_SMD:R_0603_1608Metric_Pad0.98x0.95mm_HandSolder, F.Cu at (46.6, 18.3)
- added R17: 42.2Ω, Resistor_SMD:R_0603_1608Metric_Pad0.98x0.95mm_HandSolder, F.Cu at (46.6, 20.9)
- added R18: 47kΩ, Resistor_SMD:R_0603_1608Metric_Pad0.98x0.95mm_HandSolder, F.Cu at (46.6, 23.4)
- added R19: 47kΩ, Resistor_SMD:R_0603_1608Metric_Pad0.98x0.95mm_HandSolder, F.Cu at (46.6, 25.9)
- added R20: 47kΩ, Resistor_SMD:R_0603_1608Metric_Pad0.98x0.95mm_HandSolder, F.Cu at (46.6, 28.4)
- added R21: shunt, Resistor_SMD:R_0805_2012Metric, F.Cu at (106.3, 9.43)
- added R22: 47kΩ, Resistor_SMD:R_0603_1608Metric_Pad0.98x0.95mm_HandSolder, F.Cu at (96.2, 9.21)
- added R23: 4.7kΩ, Resistor_SMD:R_0603_1608Metric_Pad0.98x0.95mm_HandSolder, F.Cu at (96.2, 11.7)
- added R24: 10kΩ, Resistor_SMD:R_0603_1608Metric_Pad0.98x0.95mm_HandSolder, F.Cu at (96.2, 14.2)
- added R25: shunt, Resistor_SMD:R_0805_2012Metric, F.Cu at (106.3, 12.4)
- added R26: 47kΩ, Resistor_SMD:R_0603_1608Metric_Pad0.98x0.95mm_HandSolder, F.Cu at (96.2, 16.7)
- added R27: 4.7kΩ, Resistor_SMD:R_0603_1608Metric_Pad0.98x0.95mm_HandSolder, F.Cu at (96.2, 19.2)
- added R28: 10kΩ, Resistor_SMD:R_0603_1608Metric_Pad0.98x0.95mm_HandSolder, F.Cu at (96.2, 21.8)
- added R29: 47kΩ, Resistor_SMD:R_0603_1608Metric_Pad0.98x0.95mm_HandSolder, F.Cu at (46.6, -6.19)
- added R30: 5.1kΩ, Resistor_SMD:R_0603_1608Metric_Pad0.98x0.95mm_HandSolder, F.Cu at (46.6, -3.68)
- added R31: 5.1kΩ, Resistor_SMD:R_0603_1608Metric_Pad0.98x0.95mm_HandSolder, F.Cu at (51.0, -13.7)
- added R32: 1kΩ, Resistor_SMD:R_0603_1608Metric_Pad0.98x0.95mm_HandSolder, F.Cu at (51.0, -11.2)
- added R33: 1kΩ, Resistor_SMD:R_0603_1608Metric_Pad0.98x0.95mm_HandSolder, F.Cu at (51.0, -8.70)
- added R34: 10kΩ, Resistor_SMD:R_0603_1608Metric_Pad0.98x0.95mm_HandSolder, F.Cu at (51.0, -6.19)
- added R35: 10kΩ, Resistor_SMD:R_0603_1608Metric_Pad0.98x0.95mm_HandSolder, F.Cu at (51.0, -3.68)
- added R36: 10kΩ, Resistor_SMD:R_0603_1608Metric_Pad0.98x0.95mm_HandSolder, F.Cu at (55.3, -13.7)
- added R37: 10kΩ, Resistor_SMD:R_0603_1608Metric_Pad0.98x0.95mm_HandSolder, F.Cu at (55.3, -11.2)
- added R38: 100kΩ, Resistor_SMD:R_0603_1608Metric_Pad0.98x0.95mm_HandSolder, F.Cu at (55.3, -8.70)
- added R39: 910kΩ, Resistor_SMD:R_0603_1608Metric_Pad0.98x0.95mm_HandSolder, F.Cu at (43.8, 61.5)
- added R40: 5.1kΩ, Resistor_SMD:R_0603_1608Metric_Pad0.98x0.95mm_HandSolder, F.Cu at (48.1, 51.5)
- added R41: 47kΩ, Resistor_SMD:R_0603_1608Metric_Pad0.98x0.95mm_HandSolder, F.Cu at (48.1, 54.0)
- added R42: 5.1kΩ, Resistor_SMD:R_0603_1608Metric_Pad0.98x0.95mm_HandSolder, F.Cu at (48.1, 56.5)
- added R43: 100kΩ, Resistor_SMD:R_0603_1608Metric_Pad0.98x0.95mm_HandSolder, F.Cu at (48.1, 59.0)
- added R44: 510kΩ, Resistor_SMD:R_0603_1608Metric_Pad0.98x0.95mm_HandSolder, F.Cu at (48.1, 61.5)
- added R45: 160kΩ, Resistor_SMD:R_0603_1608Metric_Pad0.98x0.95mm_HandSolder, F.Cu at (52.5, 51.5)
- added R46: 10kΩ, Resistor_SMD:R_0603_1608Metric_Pad0.98x0.95mm_HandSolder, F.Cu at (52.5, 54.0)
- added R47: 10kΩ, Resistor_SMD:R_0603_1608Metric_Pad0.98x0.95mm_HandSolder, F.Cu at (52.5, 56.5)
- added R48: 10kΩ, Resistor_SMD:R_0603_1608Metric_Pad0.98x0.95mm_HandSolder, F.Cu at (52.5, 59.0)
- added R49: 100Ω, Resistor_SMD:R_0603_1608Metric_Pad0.98x0.95mm_HandSolder, F.Cu at (156.0, 142.6)
- added R5: 2.2kΩ, Resistor_SMD:R_0603_1608Metric_Pad0.98x0.95mm_HandSolder, F.Cu at (19.1, 39.6)
- added R50: 100Ω, Resistor_SMD:R_0603_1608Metric_Pad0.98x0.95mm_HandSolder, F.Cu at (156.0, 145.1)
- added R51: 100Ω, Resistor_SMD:R_0603_1608Metric_Pad0.98x0.95mm_HandSolder, F.Cu at (156.0, 147.6)
- added R52: 100Ω, Resistor_SMD:R_0603_1608Metric_Pad0.98x0.95mm_HandSolder, F.Cu at (156.0, 150.1)
- added R53: 0Ω, Resistor_SMD:R_0603_1608Metric_Pad0.98x0.95mm_HandSolder, F.Cu at (123.4, 140.8)
- added R54: 0Ω, Resistor_SMD:R_0603_1608Metric_Pad0.98x0.95mm_HandSolder, F.Cu at (127.7, 133.3)
- added R55: 47kΩ, Resistor_SMD:R_0603_1608Metric_Pad0.98x0.95mm_HandSolder, F.Cu at (127.7, 135.8)
- added R56: 1kΩ, Resistor_SMD:R_0603_1608Metric_Pad0.98x0.95mm_HandSolder, F.Cu at (127.7, 138.3)
- added R57: 1kΩ, Resistor_SMD:R_0603_1608Metric_Pad0.98x0.95mm_HandSolder, F.Cu at (127.7, 140.8)
- added R58: 4.7kΩ, Resistor_SMD:R_0603_1608Metric_Pad0.98x0.95mm_HandSolder, F.Cu at (132.1, 133.3)
- added R59: 47kΩ, Resistor_SMD:R_0603_1608Metric_Pad0.98x0.95mm_HandSolder, F.Cu at (132.1, 135.8)
- added R6: 220Ω, Resistor_SMD:R_0603_1608Metric_Pad0.98x0.95mm_HandSolder, F.Cu at (19.1, 42.1)
- added R60: 5.1kΩ, Resistor_SMD:R_0603_1608Metric_Pad0.98x0.95mm_HandSolder, F.Cu at (132.1, 138.3)
- added R61: 5.1kΩ, Resistor_SMD:R_0603_1608Metric_Pad0.98x0.95mm_HandSolder, F.Cu at (132.1, 140.8)
- added R62: 1kΩ, Resistor_SMD:R_0603_1608Metric_Pad0.98x0.95mm_HandSolder, F.Cu at (289.6, 98.5)
- added R63: 1kΩ, Resistor_SMD:R_0603_1608Metric_Pad0.98x0.95mm_HandSolder, F.Cu at (289.6, 101.0)
- added R64: 1kΩ, Resistor_SMD:R_0603_1608Metric_Pad0.98x0.95mm_HandSolder, F.Cu at (289.6, 103.5)
- added R65: 1kΩ, Resistor_SMD:R_0603_1608Metric_Pad0.98x0.95mm_HandSolder, F.Cu at (289.6, 106.0)
- added R66: shunt, Resistor_SMD:R_1206_3216Metric, F.Cu at (298.0, 74.2)
- added R67: 47kΩ, Resistor_SMD:R_0603_1608Metric_Pad0.98x0.95mm_HandSolder, F.Cu at (277.7, 51.6)
- added R68: 4.7kΩ, Resistor_SMD:R_0603_1608Metric_Pad0.98x0.95mm_HandSolder, F.Cu at (277.7, 54.1)
- added R69: 4.7kΩ, Resistor_SMD:R_0603_1608Metric_Pad0.98x0.95mm_HandSolder, F.Cu at (277.7, 56.6)
- added R7: 47kΩ, Resistor_SMD:R_0603_1608Metric_Pad0.98x0.95mm_HandSolder, F.Cu at (19.1, 44.6)
- added R70: 10kΩ, Resistor_SMD:R_0603_1608Metric_Pad0.98x0.95mm_HandSolder, F.Cu at (277.7, 59.1)
- added R71: 10kΩ, Resistor_SMD:R_0603_1608Metric_Pad0.98x0.95mm_HandSolder, F.Cu at (277.7, 61.6)
- added R72: 10kΩ, Resistor_SMD:R_0603_1608Metric_Pad0.98x0.95mm_HandSolder, F.Cu at (277.7, 64.1)
- added R73: 1kΩ, Resistor_SMD:R_0603_1608Metric_Pad0.98x0.95mm_HandSolder, F.Cu at (277.7, 66.7)
- added R74: 200kΩ, Resistor_SMD:R_0603_1608Metric_Pad0.98x0.95mm_HandSolder, F.Cu at (277.7, 69.2)
- added R75: 200kΩ, Resistor_SMD:R_0603_1608Metric_Pad0.98x0.95mm_HandSolder, F.Cu at (277.7, 71.7)
- added R76: 10Ω, Resistor_SMD:R_0603_1608Metric_Pad0.98x0.95mm_HandSolder, F.Cu at (187.6, 55.2)
- added R77: 12kΩ, Resistor_SMD:R_0603_1608Metric_Pad0.98x0.95mm_HandSolder, F.Cu at (187.6, 57.8)
- added R78: 105kΩ, Resistor_SMD:R_0603_1608Metric_Pad0.98x0.95mm_HandSolder, F.Cu at (187.6, 60.3)
- added R79: 33kΩ, Resistor_SMD:R_0603_1608Metric_Pad0.98x0.95mm_HandSolder, F.Cu at (187.6, 62.8)
- added R8: 47kΩ, Resistor_SMD:R_0603_1608Metric_Pad0.98x0.95mm_HandSolder, F.Cu at (19.1, 47.1)
- added R80: 100Ω, Resistor_SMD:R_0603_1608Metric_Pad0.98x0.95mm_HandSolder, F.Cu at (187.6, 65.3)
- added R81: shunt, Resistor_SMD:R_0805_2012Metric, F.Cu at (265.7, 56.3)
- added R82: shunt, Resistor_SMD:R_0805_2012Metric, F.Cu at (265.7, 59.2)
- added R83: 47kΩ, Resistor_SMD:R_0603_1608Metric_Pad0.98x0.95mm_HandSolder, F.Cu at (248.7, 72.8)
- added R84: 47kΩ, Resistor_SMD:R_0603_1608Metric_Pad0.98x0.95mm_HandSolder, F.Cu at (248.7, 75.3)
- added R85: 4.7kΩ, Resistor_SMD:R_0603_1608Metric_Pad0.98x0.95mm_HandSolder, F.Cu at (248.7, 77.8)
- added R86: 4.7kΩ, Resistor_SMD:R_0603_1608Metric_Pad0.98x0.95mm_HandSolder, F.Cu at (248.7, 79.3)
- added R87: 10kΩ, Resistor_SMD:R_0603_1608Metric_Pad0.98x0.95mm_HandSolder, F.Cu at (248.7, 82.9)
- added R88: 10kΩ, Resistor_SMD:R_0603_1608Metric_Pad0.98x0.95mm_HandSolder, F.Cu at (253.0, 72.8)
- added R89: shunt, Resistor_SMD:R_0805_2012Metric, F.Cu at (265.7, 62.2)
- added R9: 47kΩ, Resistor_SMD:R_0603_1608Metric_Pad0.98x0.95mm_HandSolder, F.Cu at (23.4, 37.1)
- added R90: shunt, Resistor_SMD:R_0805_2012Metric, F.Cu at (265.7, 65.2)
- added R91: 47kΩ, Resistor_SMD:R_0603_1608Metric_Pad0.98x0.95mm_HandSolder, F.Cu at (253.0, 75.3)
- added R92: 47kΩ, Resistor_SMD:R_0603_1608Metric_Pad0.98x0.95mm_HandSolder, F.Cu at (252.0, 77.8)
- added R93: 4.7kΩ, Resistor_SMD:R_0603_1608Metric_Pad0.98x0.95mm_HandSolder, F.Cu at (252.0, 79.3)
- added R94: 4.7kΩ, Resistor_SMD:R_0603_1608Metric_Pad0.98x0.95mm_HandSolder, F.Cu at (253.0, 82.9)
- added R95: 10kΩ, Resistor_SMD:R_0603_1608Metric_Pad0.98x0.95mm_HandSolder, F.Cu at (257.4, 72.8)
- added R96: 10kΩ, Resistor_SMD:R_0603_1608Metric_Pad0.98x0.95mm_HandSolder, F.Cu at (257.4, 75.3)
- added R97: shunt, Resistor_SMD:R_0805_2012Metric, F.Cu at (265.7, 68.1)
- added R98: 47kΩ, Resistor_SMD:R_0603_1608Metric_Pad0.98x0.95mm_HandSolder, F.Cu at (257.4, 77.8)
- added R99: 4.7kΩ, Resistor_SMD:R_0603_1608Metric_Pad0.98x0.95mm_HandSolder, F.Cu at (257.4, 80.4)
- added SW2: Power sw, Button_Switch_SMD:SW_SPDT_PCM12, F.Cu at (262.9, 77.4)
- added TP1: AIN1, TestPoint:TestPoint_Pad_D1.5mm, F.Cu at (300.4, 98.7)
- added TP2: AIN2, TestPoint:TestPoint_Pad_D1.5mm, F.Cu at (300.4, 102.2)
- added U16: AS7343L-DLGM, panel:LGA-16_L3.0-W3.0-P0.50-BL, F.Cu at (80.1, 28.4)
- added U17: TPS7A2028DBV, panel:SOT-23-5_L2.9-W1.6-P0.95-LS2.7-BR, F.Cu at (62.4, 26.0)
- added U18: MICS-6814, panel:SENSOR_MICS-6814, F.Cu at (53.3, 14.3)
- added U19: AD7091R-4BRUZ, panel:TSSOP-20_L6.5-W4.4-P0.65-LS6.4-BL, F.Cu at (61.4, 13.8)
- added U20: H3LIS331DLTR, panel:LGA-16_L3.0-W3.0-P0.50-BL_SQ, F.Cu at (56.6, 21.3)
- added U21: MMC5983MA, panel:LGA-16_L3.0-W3.0-P0.50-BL_SQ, F.Cu at (61.0, 21.3)
- added U22: INA226, panel:VSSOP-10_L3.0-W3.0-P0.50-LS4.9-BL, F.Cu at (100.6, 24.9)
- added U23: INA226, panel:VSSOP-10_L3.0-W3.0-P0.50-LS4.9-BL, F.Cu at (105.0, 24.9)
- added U24: CH343K, panel:ESSOP-10_L4.9-W3.9-P1.0-LS6.0-TL-EP, F.Cu at (60.6, -10.7)
- added U25: TUSB321RWBR, panel:X2QFN-12_L1.6-W1.6-P0.40-TL, F.Cu at (36.5, 71.7)
- added U26: SY7072ABC, panel:SOT-23-6_L2.9-W1.6-P0.95-LS2.8-BL, F.Cu at (32.5, 72.4)
- added U27: CH9434A_C39831286, panel:QFN-48_L5.0-W5.0-P0.35-TL-EP3.7-1, B.Cu at (84.9, 44.5)
- added U28: 74LVC1G04GV, panel:SOT-353_L2.0-W1.2-P0.65-LS2.1-BL, F.Cu at (159.9, 133.1)
- added U29: 74LVC1G04GV, panel:SOT-353_L2.0-W1.2-P0.65-LS2.1-BL, F.Cu at (159.9, 136.6)
- added U30: 74LVC1G04GV, panel:SOT-353_L2.0-W1.2-P0.65-LS2.1-BL, F.Cu at (159.9, 140.1)
- added U31: 74LVC1G04GV, panel:SOT-353_L2.0-W1.2-P0.65-LS2.1-BL, F.Cu at (159.9, 143.6)
- added U32: E28-2G4M27SX, panel:E22-400M22S, B.Cu at (147.3, 111.3)
- added U33: SIM7080G, panel:XCVR_SIM7080G, F.Cu at (129.6, 91.4)
- added U34: RS0102YH8, panel:SOT-23-8_L3.0-W1.7-P0.65-LS2.8-BL, F.Cu at (123.6, 151.1)
- added U35: MFF2-SIM, Package_DFN_QFN:DFN-8-1EP_6x5mm_P1.27mm_EP2x2mm, F.Cu at (125.9, 145.4)
- added U36: TPS7A2028DBV, panel:SOT-23-5_L2.9-W1.6-P0.95-LS2.7-BR, F.Cu at (304.5, 105.8)
- added U37: AD7799BRUZ-REEL, panel:TSSOP-16_L5.0-W4.4-P0.65-LS6.4-BL, F.Cu at (295.5, 101.1)
- added U38: INA226, panel:VSSOP-10_L3.0-W3.0-P0.50-LS4.9-BL, F.Cu at (293.1, 76.1)
- added U39: XT30AW-M.G.Y, panel:CONN-TH_XT30AW-M.G.Y, F.Cu at (212.9, 47.5)
- added U40: AP64501SP-13, panel:SOIC-8-1EP_3.9x4.9mm_P1.27mm_EP2.95x4.9mm_Mask2.71x3.4mm_ThermalVias_BigVias, F.Cu at (194.0, 52.3)
- added U41: INA226, panel:VSSOP-10_L3.0-W3.0-P0.50-LS4.9-BL, F.Cu at (243.1, 51.3)
- added U42: INA226, panel:VSSOP-10_L3.0-W3.0-P0.50-LS4.9-BL, F.Cu at (247.4, 51.3)
- added U43: INA226, panel:VSSOP-10_L3.0-W3.0-P0.50-LS4.9-BL, F.Cu at (251.7, 51.3)
- added U44: INA226, panel:VSSOP-10_L3.0-W3.0-P0.50-LS4.9-BL, F.Cu at (256.0, 51.3)
- added U45: INA226, panel:VSSOP-10_L3.0-W3.0-P0.50-LS4.9-BL, F.Cu at (260.3, 51.3)
- added U46: INA226, panel:VSSOP-10_L3.0-W3.0-P0.50-LS4.9-BL, F.Cu at (314.9, 65.5)
- added U47: INA226, panel:VSSOP-10_L3.0-W3.0-P0.50-LS4.9-BL, F.Cu at (319.2, 65.5)
- added U48: TCA9546APW, panel:TSSOP-16_L5.0-W4.4-P0.65-LS6.4-BL, F.Cu at (-219.9, -52.6)
- added U49: BME280, panel:BME280_PSON65P250X250X100-8N, F.Cu at (-238.9, -62.5)
- added U50: VEML7700-TT, panel:XDCR_VEML7700-TT, F.Cu at (-237.6, -68.8)
- added U51: BME280, panel:BME280_PSON65P250X250X100-8N, F.Cu at (-238.9, -58.4)
- added U52: VEML7700-TT, panel:XDCR_VEML7700-TT, F.Cu at (-231.9, -68.8)
- added U53: BME280, panel:BME280_PSON65P250X250X100-8N, F.Cu at (-238.9, -54.2)
- added U54: VEML7700-TT, panel:XDCR_VEML7700-TT, F.Cu at (-226.2, -68.8)
- added U55: BME280, panel:BME280_PSON65P250X250X100-8N, F.Cu at (-238.9, -50.1)
- added U56: VEML7700-TT, panel:XDCR_VEML7700-TT, F.Cu at (-220.6, -68.8)
- added U57: MAX5026EUT+T, panel:SOT-23-6_L2.9-W1.6-P0.95-LS2.8-BL, F.Cu at (-204.8, -27.5)
- added U58: ADS8331IPWR, panel:TSSOP-24_L7.8-W4.4-P0.65-LS6.4-BL, F.Cu at (-197.1, -38.8)
- added U59: DAC124S085CIMM/NOPB, panel:VSSOP-10_L3.0-W3.0-P0.50-LS4.9-BL, F.Cu at (-194.9, -30.9)
- added U60: TPS7A2028DBV, panel:SOT-23-5_L2.9-W1.6-P0.95-LS2.7-BR, F.Cu at (-194.8, -25.3)
- added U61: OPA365AIDBVR, panel:SOT-23-5_L3.0-W1.7-P0.95-LS2.8-BR, F.Cu at (-196.4, -56.4)
- added U62: OPA365AIDBVR, panel:SOT-23-5_L3.0-W1.7-P0.95-LS2.8-BR, F.Cu at (-196.4, -52.1)
- added U63: TLV3501AIDBV, panel:SOT-23-6_L2.9-W1.6-P0.95-LS2.9-BL, F.Cu at (-209.3, -49.6)
- added U64: LM27762DSSR, panel:WSON-12_L3.0-W2.0-P0.50-BL-EP, F.Cu at (-233.5, -22.8)
- added U65: OPA858IDSGR, Package_SON:Texas_DSG0008A_WSON-8-1EP_2x2mm_P0.5mm_EP0.9x1.6mm, F.Cu at (-220.3, -30.2)
- added U66: OPA365AIDBVR, panel:SOT-23-5_L3.0-W1.7-P0.95-LS2.8-BR, F.Cu at (-238.6, -19.7)
- added U67: TLV3501AIDBV, panel:SOT-23-6_L2.9-W1.6-P0.95-LS2.9-BL, F.Cu at (-219.8, -34.2)
- added U68: RS0102YH8, panel:SOT-23-8_L3.0-W1.7-P0.65-LS2.8-BL, F.Cu at (-83.8, -33.5)
- added U69: RS0102YH8, panel:SOT-23-8_L3.0-W1.7-P0.65-LS2.8-BL, F.Cu at (-79.3, -33.5)
- added U70: TXB0104RUTR, panel:UQFN-12_L2.0-W1.7-P0.40-BL, F.Cu at (-69.5, -51.7)
- added U71: TPS7A2028DBV, panel:SOT-23-5_L2.9-W1.6-P0.95-LS2.7-BR, F.Cu at (-70.1, -37.7)
- added U72: TPS7A2028DBV, panel:SOT-23-5_L2.9-W1.6-P0.95-LS2.7-BR, F.Cu at (-70.1, -33.2)
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Connections:
- net /Display/ghgh renamed Net-(J1-Pin_14)
- IC1 pad 1: GND -> /Panel1_MCU/I2C0_SCL
- IC1 pad 10: GND -> /Panel1_MCU/I2C_Sensors/3.3V
- IC1 pad 11: GND -> /Panel1_MCU/I2C_Sensors/3.3V
- IC1 pad 12: GND -> /Panel1_MCU/I2C_Sensors/3.3V
- IC1 pad 2: GND -> /Panel1_MCU/I2C0_SDA
- IC1 pad 3: GND -> unconnected-(IC1-INT-Pad3)
- IC1 pad 4: GND -> unconnected-(IC1-N.C._1-Pad4)
- IC1 pad 5: GND -> /Panel1_MCU/I2C_Sensors/3.3V
- IC1 pad 6: unconnected-(IC1-RXEN-Pad6) -> GND
- IC1 pad 7: unconnected-(IC1-TXEN-Pad7) -> GND
- IC1 pad 9: unconnected-(IC1-VCC-Pad9) -> GND
- IC2 pad 1: unconnected-(IC2-SCL-Pad1) -> GND
- IC2 pad 10: unconnected-(IC2-VDDH-Pad10) -> GND
- IC2 pad 11: unconnected-(IC2-RES_N-Pad11) -> GND
- IC2 pad 12: unconnected-(IC2-VDDIO-Pad12) -> GND
- IC2 pad 2: unconnected-(IC2-SDA-Pad2) -> GND
- IC2 pad 3: unconnected-(IC2-INT-Pad3) -> GND
- IC2 pad 4: unconnected-(IC2-N.C._1-Pad4) -> GND
- IC2 pad 5: unconnected-(IC2-VDD-Pad5) -> GND
- IC2 pad 6: unconnected-(IC2-VSS_1-Pad6) -> /Panel2_COM/900MHZ_RXEN
- IC2 pad 7: unconnected-(IC2-VSS_2-Pad7) -> /Panel2_COM/900MHZ_TXEN
- IC2 pad 8: unconnected-(IC2-N.C._2-Pad8) -> /Panel2_COM/900MHZ_DIO2
- IC2 pad 9: unconnected-(IC2-VSS_3-Pad9) -> /Panel2_COM/Radio_900Mhz_PWR
- MT1 pad 1: unconnected-(MT1-AP_SDO/AP_AD0-Pad1) -> /Panel1_MCU/LP_MISO
- MT1 pad 10: Net-(MT1-RESV-Pad10) -> unconnected-(MT1-RESV-Pad10)_1
- MT1 pad 11: Net-(MT1-RESV-Pad10) -> unconnected-(MT1-RESV-Pad10)_3
- MT1 pad 12: unconnected-(MT1-AP_CS-Pad12) -> /Panel1_MCU/ICM_LP_CS
- MT1 pad 13: unconnected-(MT1-AP_SCL/AP_SCLK-Pad13) -> /Panel1_MCU/LP_SCK
- MT1 pad 14: unconnected-(MT1-AP_SDA/AP_SDIO/AP_SDI-Pad14) -> /Panel1_MCU/LP_MOSI
- MT1 pad 2: Net-(MT1-RESV-Pad10) -> unconnected-(MT1-RESV-Pad10)
- MT1 pad 3: Net-(MT1-RESV-Pad10) -> unconnected-(MT1-RESV-Pad10)_2
- MT1 pad 5: unconnected-(MT1-VDDIO-Pad5) -> /Panel1_MCU/Sensors_3.3V
- MT1 pad 6: unconnected-(MT1-GND-Pad6) -> GND
- MT1 pad 7: unconnected-(MT1-FSYNC-Pad7) -> /Panel1_MCU/LEPTON_VSYNC
- MT1 pad 8: unconnected-(MT1-VDD-Pad8) -> /Panel1_MCU/Sensors_3.3V
- R1 pad 2: /Display/dffgdgdxxa -> /Panel1_MCU/Sensors_3.3V
- R2 pad 1: /Display/hghdh -> /Panel1_MCU/I2C0_SCL
- R2 pad 2: /Display/sfaddsQA -> /Panel1_MCU/Standby_3.3V
- R3 pad 1: /SiPM_detectors/ghgh -> /Panel1_MCU/I2C0_SDA
- R3 pad 2: /SiPM_detectors/dffgdgdxxa -> /Panel1_MCU/Standby_3.3V
- R4 pad 1: /SiPM_detectors/hghdh -> /Panel1_MCU/I2C1_SCL
- R4 pad 2: /SiPM_detectors/sfaddsQA -> /Panel1_MCU/Standby_3.3V
- U1 pad 1: unconnected-(U1-VDD-Pad1) -> GND
- U1 pad 15: unconnected-(U1-VIN1-Pad15) -> GND
- U1 pad 17: GND -> /Panel1_MCU/LP_I2C_SCL
- U1 pad 18: unconnected-(U1-SDI-Pad18) -> /Panel1_MCU/LP_I2C_SDA
- U1 pad 19: unconnected-(U1-SDO-Pad19) -> /Panel1_MCU/LP_MISO
- U1 pad 20: unconnected-(U1-SCLK-Pad20) -> /Panel1_MCU/LP_MOSI
- U1 pad 22: unconnected-(U1-VDRIVE-Pad22) -> /Panel1_MCU/LP_SCK
- U1 pad 23: unconnected-(U1-~{CS}-Pad23) -> /Panel1_MCU/LP_CS_DEMUX_A
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Other:
- board outline added: 173.2 x 52.5 mm
- copper layers 2 -> 4
