File: Circuit/CanSat_V2/CanSat.kicad_sch (KiCad schematic)
At the start: 20 parts, among them IC1 E22-900M22S, IC2 ZMOD4410AI1V, J1 FLIR_Lepton_Molex_1050281001, SW1 SKRHABE010, U1 AD7091R-8BCPZ-RL7, U10 SCD41-D-R2, U11 SGP41-D-R4, U12 SHT41-AD1B-R2, U13 SIM7080G, U14 STC31-C-R3, U15 VEML7700-TT, U2 AS7331-AQFM, U3 ADS1220IPWR, U4 BME280, U5 BME688, U6 ESP32-P4-Module, U7 LC86G, U8 MICS-6814, U9 RadNano

Commit message: first cansat V2 commit
Parts:
- removed IC1: E22-900M22S, panel:E22-900M22S, symbol panel:E22-900M22S
- removed IC2: ZMOD4410AI1V, panel:ZMOD4510AI1V, symbol panel:ZMOD4410AI1V
- removed J1: FLIR_Lepton_Molex_1050281001, panel:flir_CONN_1050282031_MOL, symbol panel:FLIR_Lepton_Molex_1050281001
- removed MT1: ICM-42670-P, panel:XDCR_ICM-42670-P, symbol panel:ICM-42670-P
- removed SW1: SKRHABE010, panel:SKRHABE010_ALPS, symbol panel:SKRHABE010
- removed U1: AD7091R-8BCPZ-RL7, panel:SOP65P640X120-24N, symbol panel:AD7091R-8BCPZ-RL7
- removed U10: SCD41-D-R2, panel:XDCR_SCD41-D-R2, symbol panel:SCD41-D-R2
- removed U11: SGP41-D-R4, panel:XDCR_SGP41-D-R4, symbol panel:SGP41-D-R4
- removed U12: SHT41-AD1B-R2, panel:STC42A, symbol panel:SHT41-AD1B-R2
- removed U13: SIM7080G, panel:XCVR_SIM7080G, symbol panel:SIM7080G
- removed U14: STC31-C-R3, panel:STC42A, symbol panel:STC31-C-R3
- removed U15: VEML7700-TT, panel:XDCR_VEML7700-TT, symbol panel:VEML7700-TT
- removed U2: AS7331-AQFM, panel:PQFN50P365X260X119-16N, symbol panel:AS7331-AQFM
- removed U3: ADS1220IPWR, panel:SOP65P640X120-16N, symbol panel:ADS1220IPWR
- removed U4: BME280, panel:BME280_PSON65P250X250X100-8N, symbol panel:BME280
- removed U5: BME688, panel:IC_BME688, symbol panel:BME688
- removed U6: ESP32-P4-Module, panel:ESP32-P4, symbol panel:ESP32-P4-Module
- removed U7: LC86G, panel:XCVR_LC86G, symbol panel:LC86G
- removed U8: MICS-6814, panel:SENSOR_MICS-6814, symbol panel:MICS-6814
- removed U9: RadNano, panel:RadNano, symbol panel:RadNano
Other:
- removed sheet 3_SX12xx_Series_radio
- removed sheet Display
- removed sheet FLIR_Lepton_3.1R
- removed sheet GPS
- removed sheet LTE_modem
- removed sheet Processor
- removed sheet SiPM_detectors
- removed sheet gas_sensors
- removed sheet psu
- added sheet Panel1_MCU (Panel1_MCU.kicad_sch)
- added sheet Panel2_COM (Panel2_COM.kicad_sch)
- added sheet Panel3_GLM-PSU (Panel3_GLM-PSU.kicad_sch)
- added sheet Panel4_BAT_Plate (Panel4_BAT_Plate.kicad_sch)
- added sheet Panel5_FLIR (Panel5_FLIR.kicad_sch)
- note added: "python -m easyeda2kicad --full --lcsc_id C19268026 --output "D:\Data\T.E.E.M.O\Circuit\CanSat_V2\panel"
