File: Circuit/CanSat_V2/GPS.kicad_sch (KiCad schematic)
At the start: 0 parts

Commit message: first cansat V2 commit
Parts:
- added C3: 22uF, Capacitor_SMD:C_1210_3225Metric, symbol Device:C
- added C4: 100nF, Capacitor_SMD:C_0603_1608Metric_Pad1.08x0.95mm_HandSolder, symbol Device:C
- added D3: LED, LED_SMD:LED_0603_1608Metric_Pad1.05x0.95mm_HandSolder, symbol Device:LED
- added R11: 10kΩ, Resistor_SMD:R_0603_1608Metric_Pad0.98x0.95mm_HandSolder, symbol Device:R
- added R12: 220Ω, Resistor_SMD:R_0603_1608Metric_Pad0.98x0.95mm_HandSolder, symbol Device:R
- added U5: LC86G, panel:XCVR_LC86G, symbol panel:LC86G
Connections:
- new net: D3.2 (A), R12.1
- new net: R12.2, U5.6 (1PPS)
- new net: R11.2, U5.10 (~{RESET})
- new net: U5.7 (RESERVED), U5.9 (RESERVED)
- new net 3.3V: C3.1, C4.1, R11.1, U5.4 (VCC), U5.5 (V_BCKP)
- new net GND: C3.2, C4.2, D3.1 (K), U5.12 (GND), U5.13 (GND), U5.14 (GND), U5.15 (GND), U5.16 (GND), U5.17 (GND), U5.18 (GND), U5.19 (GND), U5.20 (GND), U5.21 (GND), U5.22 (GND), U5.23 (GND), U5.24 (GND), U5.25 (GND), U5.26 (GND), U5.27 (GND), U5.28 (GND), U5.29 (GND), U5.3 (GND), U5.30 (GND), U5.31 (GND), U5.32 (GND), U5.33 (GND), U5.34 (GND), U5.35 (GND), U5.36 (GND)
- new net RX: U5.2 (TXD)
- new net TX: U5.1 (RXD)
- no-connect marks 0 -> 2
