File: Circuit/CanSat_V2/LTE_modem.kicad_sch (KiCad schematic)
At the start: 0 parts

Commit message: first cansat V2 commit
Parts:
- added C42, C43, C44, C45: -, Capacitor_SMD:C_0402_1005Metric_Pad0.74x0.62mm_HandSolder, symbol Device:C
- added C46, C47, C50: 100nF, Capacitor_SMD:C_0603_1608Metric_Pad1.08x0.95mm_HandSolder, symbol Device:C
- added C48, C49: 22uF, Capacitor_SMD:C_1210_3225Metric, symbol Device:C_Polarized
- added D6, D7: ESD5311X-2/TR, Diode_SMD:D_0402_1005Metric_Pad0.77x0.64mm_HandSolder, symbol panel:ESD5311X-2_TR
- added D8, D9: LED, LED_SMD:LED_0603_1608Metric_Pad1.05x0.95mm_HandSolder, symbol Device:LED
- added J7, J8: U-Fl-IPEX, panel:IPEX-SMD_4P-L2.6-W2.6-LS3.1, symbol Connector:Conn_Coaxial
- added J9: USB_C, Connector_USB:USB_C_Receptacle_Palconn_UTC16-G, symbol Connector:USB_C_Receptacle_USB2.0_16P
- added Q8: BC817, Package_TO_SOT_SMD:SOT-23, symbol Simulation_SPICE:NPN
- added R53, R54: 0Ω, Resistor_SMD:R_0603_1608Metric_Pad0.98x0.95mm_HandSolder, symbol Device:R
- added R55, R59: 47kΩ, Resistor_SMD:R_0603_1608Metric_Pad0.98x0.95mm_HandSolder, symbol Device:R
- added R56, R57: 1kΩ, Resistor_SMD:R_0603_1608Metric_Pad0.98x0.95mm_HandSolder, symbol Device:R
- added R58: 4.7kΩ, Resistor_SMD:R_0603_1608Metric_Pad0.98x0.95mm_HandSolder, symbol Device:R
- added R60, R61: 5.1kΩ, Resistor_SMD:R_0603_1608Metric_Pad0.98x0.95mm_HandSolder, symbol Device:R
- added U33: SIM7080G, panel:XCVR_SIM7080G, symbol panel:SIM7080G
- added U34: RS0102YH8, panel:SOT-23-8_L3.0-W1.7-P0.65-LS2.8-BL, symbol panel:RS0102YH8
- added U35: MFF2-SIM, Package_DFN_QFN:DFN-8-1EP_6x5mm_P1.27mm_EP2x2mm, symbol panel:SIM_MFF2
Connections:
- new net: D8.2 (A), R56.2
- new net: C45.2, D7.1, J8.1 (In), R54.2
- new net: Q8.1 (B), R58.1
- new net: Q8.3 (C), R55.2, U33.39 (PWRKEY)
- new net: D9.2 (A), R57.2
- new net: J9.A5 (CC1), R60.2
- new net: C44.1, D6.1, J7.1 (In), R53.2
- new net: J9.B5 (CC2), R61.2
- new net: U33.1 (UART1_TXD), U34.6 (A2)
- new net: U33.2 (UART1_RXD), U34.7 (A1)
- new net 1.8V: R55.1, U33.40 (VDD_EXT), U34.4 (OE), U34.8 (VCCA)
- new net GND: C42.2, C43.1, C44.2, C45.1, C46.2, C47.2, C48.2, C49.2, C50.2, D6.2, D7.2, D8.1 (K), D9.1 (K), J7.2 (Ext), J8.2 (Ext), J9.A1 (GND), J9.A12 (GND), J9.B1 (GND), J9.B12 (GND), J9.S1 (SHIELD), Q8.2 (E), R59.1, R60.1, R61.1, U33.13 (GND), U33.19 (GND), U33.21 (GND), U33.27 (GND), U33.30 (GND), U33.31 (GND), U33.33 (GND), U33.36 (GND), U33.37 (GND), U33.45 (GND), U33.63 (GND), U33.66 (GND), U33.67 (GND), U33.69 (GND), U33.70 (GND), U33.71 (GND), U33.72 (GND), U33.73 (GND), U33.74 (GND), U33.75 (GND), U33.76 (GND), U33.77 (GND), U33.8 (GND), U34.5 (GND), U35.5 (GND), U35.9 (GND)
- new net NETLIGHT: R56.1, U33.41 (NETLIGHT)
- new net PWRKEY: R58.2
- new net RF_GNSS: C43.2, R54.1, U33.68 (GNSS_ANT)
- new net RF_LTE: C42.1, R53.1, U33.32 (RF_ANT)
- new net RX: U34.3 (B2)
- new net SIM_CLK: U33.16 (SIM_CLK), U35.3 (CLK)
- new net SIM_DATA: U33.15 (SIM_DATA), U35.7 (I/O)
- new net SIM_RST: U33.17 (SIM_RST), U35.2 (RST)
- new net SIM_VDD: C50.1, U33.18 (SIM_VDD), U35.1 (VCC)
- new net STATUS: R57.1, U33.42 (STATUS)
- new net TX: U34.2 (B1)
- new net USB_D+: J9.A6 (D+), J9.B6 (D+), U33.25 (USB_DP)
- new net USB_D-: J9.A7 (D-), J9.B7 (D-), U33.26 (USB_DM)
- new net VBAT: C47.1, C48.1, C49.1, U33.34 (VBAT), U33.35 (VBAT), U34.1 (VCCB)
- new net VBUS: C46.1, J9.A4 (VBUS), J9.A9 (VBUS), J9.B4 (VBUS), J9.B9 (VBUS), R59.2, U33.24 (USB_VBUS)
- no-connect marks 0 -> 30
Other:
- note added: "Level Shifter"
- note added: "Level Shifter (PowerKey)"
- note added: "RF_OUT"
- note added: "SIMCOM Update Port"
- note added: "Simcard"
- note added: "Status LEDs"
