File: Circuit/CanSat_V2/SiPM_detectors.kicad_sch (KiCad schematic)
At the start: 0 parts

Commit message: first cansat V2 commit
Parts:
- added C112, C113, C116, C117: 4.7uF, Capacitor_SMD:C_1206_3216Metric, symbol Device:C
- added C114, C115: 100nF, Capacitor_SMD:C_0603_1608Metric_Pad1.08x0.95mm_HandSolder, symbol Device:C
- added D11: BAT54J, Diode_SMD:D_SOD-323_HandSoldering, symbol Diode:BAT54J
- added FB1, FB2: FerriteBead_Small, Diode_SMD:D_0805_2012Metric, symbol Device:FerriteBead_Small
- added L3: 47uh, Diode_SMD:D_0805_2012Metric, symbol Device:L_Small
- added R114: 68kΩ, Resistor_SMD:R_0603_1608Metric_Pad0.98x0.95mm_HandSolder, symbol Device:R
- added R115: 154kΩ, Resistor_SMD:R_0603_1608Metric_Pad0.98x0.95mm_HandSolder, symbol Device:R
- added R116: 6,65kΩ, Resistor_SMD:R_0603_1608Metric_Pad0.98x0.95mm_HandSolder, symbol Device:R
- added R117: 470kΩ, Resistor_SMD:R_0603_1608Metric_Pad0.98x0.95mm_HandSolder, symbol Device:R
- added R118: 39kΩ, Resistor_SMD:R_0603_1608Metric_Pad0.98x0.95mm_HandSolder, symbol Device:R
- added U57: MAX5026EUT+T, panel:SOT-23-6_L2.9-W1.6-P0.95-LS2.8-BL, symbol panel:MAX5026EUT+T
- added U58: ADS8331IPWR, panel:TSSOP-24_L7.8-W4.4-P0.65-LS6.4-BL, symbol panel:ADS8331IPWR
- added U59: DAC124S085CIMM/NOPB, panel:VSSOP-10_L3.0-W3.0-P0.50-LS4.9-BL, symbol panel:DAC124S085CIMM_NOPB
- added U60: TPS7A2028DBV, panel:SOT-23-5_L2.9-W1.6-P0.95-LS2.7-BR, symbol Regulator_Linear:TPS7A20xxxDBV
Connections:
- new net: R114.2, R115.2, R116.1, U57.3 (FB)
- new net: D11.2 (A), L3.1, U57.6 (LX)
- new net: U58.21 (ADCIN), U58.22 (MUXOUT)
- new net 2.8V: C117.1, U58.18 (REF+), U59.7 (VREFIN), U60.5 (OUT)
- new net COMP: R114.1, U59.2 (VOUTA)
- new net GND: C112.2, C113.2, C114.2, C115.2, C116.2, C117.2, R116.2, R118.2, U57.1 (PGND), U57.2 (GND), U58.14 (DGND), U58.15 (~{CONVST}), U58.19 (REF-), U58.20 (AGND), U58.23 (COM), U59.6 (GND), U60.2 (GND)
- new net Gamma Ch/+3.3V: FB1.1
- new net Gamma Ch/+30V: C113.1, C114.1, D11.1 (K), R115.1, R117.1
- new net Gamma_ADC: U58.24 (IN0)
- new net Gamma_Thres: U59.4 (VOUTC)
- new net MAX_COMP: C115.1, R117.2, R118.1, U58.3 (IN3)
- new net Muon_Thres: U59.3 (VOUTB)
- new net Müon Ch/+3.3V: FB2.1
- new net Müon_ADC: U58.1 (IN1)
- new net NTC1: U58.2 (IN2)
- new net SPI_CS_1: U59.9 (~{SYNC})
- new net SPI_CS_2: U58.11 (FS/~{CS})
- new net SPI_MISO: U58.13 (SDO)
- new net SPI_MOSI: U58.12 (SDI), U59.8 (DIN)
- new net SPI_SCK: U58.10 (SCLK), U59.10 (SCLK)
- new net SiPM_3.3V: C112.1, C116.1, FB1.2, FB2.2, L3.2, U57.4 (~{SHDN}), U57.5 (VCC), U58.16 (VBD), U58.17 (VA), U58.8 (~{RESET}), U59.1 (VA), U60.1 (IN), U60.3 (EN)
- no-connect marks 0 -> 6
Other:
- added sheet Gamma Ch (SiPM_2.kicad_sch)
- added sheet Müon Ch (SiPM_1.kicad_sch)
